Commit message: urdf bag fixed

File: example/urdf/plug.urdf (robot description, URDF)
Before this commit: robot plug, 2 links, 1 joints
Links:
- link plug_link: geometry collision mesh filename=meshes/plug/plug.stl scale=0.001 0.001 0.001; visual mesh filename=meshes/plug/plug.stl scale=0.001 0.001 0.001

File: example/urdf/socket.urdf (robot description, URDF)
Before this commit: robot socket, 2 links, 1 joints
Links:
- link socket_link: geometry collision mesh filename=meshes/socket/socket.stl scale=0.001 0.001 0.001; visual mesh filename=meshes/socket/socket.stl scale=0.001 0.001 0.001
